File: Receiver_Out/Diff_In.sch (KiCad schematic (older format))
At the start: 4 parts, among them J7 RJ45, U3 AM26C32IN

Commit message: fixed the schematic, to match the PCB
Parts:
- U3: symbol AM26C32IN:AM26C32IN -> Receiver_Out-rescue:AM26C32IN-AM26C32IN
Changed lines of the file:
@@
 $EndComp
 $Comp
-L AM26C32IN:AM26C32IN U3
+L Receiver_Out-rescue:AM26C32IN-AM26C32IN U3
 U 1 1 5E069391
 P 4455 4160
+AR Path="/5E069391" Ref="U3"  Part="1"
+AR Path="/5E06688B/5E069391" Ref="U3"  Part="1"
 F 0 "U3" H 5955 4547 60  0000 C CNN
 F 1 "AM26C32IN" H 5955 4441 60  0000 C CNN
