File: PB_16_Mini/PB_16.sch (KiCad schematic (older format))
At the start: 23 parts, among them J1 USB, J2 OLED Conn, J3 GPIO Header, J4 RTC Conn, J5 Power In, J6 VIN_Voltage, J7 Output Header, SW1 OLED Select, SW4 Enter BTN, SW5 Down BTN, U1 LM7805, U4 24LC256

Commit message: Added PDF of most of the Schematics
Other:
- moved on the sheet: C1, C2, C3, C6, D1, D2, F1, F2, J2, J3, J4, J5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

Commit message: fix DMX1 pins backwards
Parts:
- J1: symbol Connector:USB_A -> PB_16-rescue:USB_A-Connector
Changed lines of the file:
@@
 USB_D-
 $Comp
-L Connector:USB_A J1
+L PB_16-rescue:USB_A-Connector J1
 U 1 1 5D4E8733
 P 1695 2465
