File: PB_16_Mini/PocketBeagle.kicad_sch (KiCad schematic)
At the start: 2 parts, among them U2 POCKETBEAGLE-SC-569

Commit message: working on v4
Connections:
- net OUT1: now also U2.P2_34 (PRU0_5); no longer U2.P2_22 (GPIO_46)
- net OUT10: now also U2.P2_8 (GPIO_60); no longer U2.P2_25 (SPI1_MOSI)
- net OUT11: now also U2.P2_5 (UART4_RX); no longer U2.P2_27 (SPI1_MISO)
- net OUT12: now also U2.P2_6 (GPIO_57); no longer U2.P2_33 (GPIO_45)
- net OUT13: now also U2.P2_4 (GPIO_58); no longer U2.P1_29 (PRU0_7)
- net OUT14: now also U2.P2_3 (GPIO_23); no longer U2.P2_34 (PRU0_5)
- net OUT15: now also U2.P2_2 (GPIO_59); no longer U2.P2_30 (PRU0_3)
- net OUT16: now also U2.P2_1 (PWM1_A); no longer U2.P1_33 (PRU0_1)
- net OUT2: now also U2.P2_32 (PRU0_2); no longer U2.P2_18 (GPIO_47)
- net OUT3: now also U2.P2_30 (PRU0_3); no longer U2.P2_10 (GPIO_52)
- net OUT4: now also U2.P2_28 (PRU0_6); no longer U2.P2_8 (GPIO_60)
- net OUT5: now also U2.P2_24 (GPIO_48); no longer U2.P2_6 (GPIO_57)
- net OUT6: now also U2.P2_22 (GPIO_46); no longer U2.P2_4 (GPIO_58)
- net OUT7: now also U2.P2_20 (GPIO_64); no longer U2.P2_2 (GPIO_59)
- net OUT8: now also U2.P2_18 (GPIO_47); no longer U2.P2_1 (PWM1_A)
- net OUT9: now also U2.P2_7 (UART4_TX); no longer U2.P2_24 (GPIO_48)
- net TXD1: now also U2.P2_9 (I2C1_SCL); no longer U2.P2_32 (PRU0_2)
- net TXD2: now also U2.P1_10 (SPI0_MISO); no longer U2.P1_36 (PWM0_A)
- net OUT19: now reaches U2.P2_29 (SPI1_CLK)
- net OUT20: now reaches U2.P2_31 (SPI1_CS)
- net OUT18: now reaches U2.P2_35 (AIN5/GPIO86)
- new net OUT17: U2.P2_33 (GPIO_45)
- no-connect marks 35 -> 31
Other:
- title: PB 16 Min -> PB 16 Mini
- moved on the sheet: U2A, U2B
