File: PB_16_Mini/Serial.kicad_sch (KiCad schematic)
At the start: 8 parts, among them J10 DMX2 RJ45, J9 DMX1 RJ45, SW2 DMX_Renard_Select, SW3 DMX_LOR_Select, U3 UA9638CP

Commit message: working on v4
Parts:
- removed J10: DMX2 RJ45, Scotts:RJ45_Amphenol_54602-x08_Horizontal, symbol Connector:RJ45
- removed SW2: DMX_Renard_Select, Button_Switch_THT:SW_CuK_JS202011CQN_DPDT_Straight, symbol Switch:SW_DPDT_x2
- removed SW3: DMX_LOR_Select, Button_Switch_THT:SW_CuK_JS202011CQN_DPDT_Straight, symbol Switch:SW_DPDT_x2
- added J8: DMX2, TerminalBlock_Phoenix:TerminalBlock_Phoenix_MKDS-1,5-3_1x03_P5.00mm_Horizontal, symbol Connector:Screw_Terminal_01x03
Connections:
- net DMX1+: now also J9.1
- net DMX1-: now also J9.2
- net DMX2+: now also J8.1 (Pin_1)
- net DMX2-: now also J8.2 (Pin_2)
- net GND: now also J8.3 (Pin_3)
- net 9V: no longer names the net of J9.3
- no-connect marks 3 -> 1
Other:
- title: PB 16 Min -> PB 16 Mini
- moved on the sheet: C5, J9, R3, U3B
