File: 16_Expansion_SMD/Output1_8.sch (KiCad schematic (older format))
At the start: 20 parts, among them J1 String1, J2 String2, J3 String3, J4 String4, J5 String5, J6 String6, J7 String7, J8 String8, U1 74HC245

Commit message: added BOM and Position file for SMD assembly
Parts:
- C1: Digi-Key_PN 478-7336-1-ND -> 478-1395-1-ND; LCSC (none) -> C49678; MPN SR215C104KARTR1 -> 08055C104KAT2A
- U1: Digi-Key_PN (none) -> 296-8279-1-ND; LCSC (none) -> C5625; MPN (none) -> SN74HC245PWR
Changed lines of the file:
@@
 F 2 "Capacitor_SMD:C_0805_2012Metric_Pad1.15x1.40mm_HandSolder" H 5138 3800 50  0001 C CNN
 F 3 "~" H 5100 3950 50  0001 C CNN
-F 4 "478-7336-1-ND" H -1680 -380 50  0001 C CNN "Digi-Key_PN"
-F 5 "SR215C104KARTR1" H -1680 -380 50  0001 C CNN "MPN"
+F 4 "478-1395-1-ND" H -1680 -380 50  0001 C CNN "Digi-Key_PN"
+F 5 "08055C104KAT2A" H -1680 -380 50  0001 C CNN "MPN"
+F 6 "C49678" H 5100 3950 50  0001 C CNN "LCSC"
 	1    5100 3950
 	1    0    0    -1
@@
 F 2 "Package_SO:SOIC-20W_7.5x12.8mm_P1.27mm" H 4630 4990 50  0001 C CNN
 F 3 "http://www.ti.com/lit/gpn/sn74HC245" H 4630 4990 50  0001 C CNN
+F 4 "296-8279-1-ND" H 4630 4990 50  0001 C CNN "Digi-Key_PN"
+F 5 "C5625" H 4630 4990 50  0001 C CNN "LCSC"
+F 6 "SN74HC245PWR" H 4630 4990 50  0001 C CNN "MPN"
 	1    4630 4990
 	1    0    0    -1
