File: BBB_16_Expansion/PocketBeagle.kicad_sch (KiCad schematic)
At the start: 3 parts, among them SW1 PWR_BUTTON, U1 BEAGLEBONEBLACK

Commit message: added Gerbers and BOM
Parts:
- C4: Field4 (none) -> C49678; Field5 (none) -> CL21F104ZBCNNNC; Field6 (none) -> 1276-1007-1-ND; Field7 (none) -> C49678; Field8 (none) -> CL21F104ZBCNNNC; LCSC C49678 -> 1276-1007-1-ND; MPN CL21F104ZBCNNNC -> C49678
Changed lines of the file:
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@@
       (effects (font (size 1.27 1.27)) hide)
     )
-    (property "MPN" "CL21F104ZBCNNNC" (id 5) (at 43.18 66.04 0)
+    (property "MPN" "C49678" (id 5) (at 43.18 66.04 0)
       (effects (font (size 1.27 1.27)) hide)
     )
-    (property "LCSC" "C49678" (id 6) (at 43.18 66.04 0)
+    (property "LCSC" "1276-1007-1-ND" (id 6) (at 43.18 66.04 0)
       (effects (font (size 1.27 1.27)) hide)
     )
+    (property "Field4" "C49678" (id 7) (at 43.18 66.04 0)
+      (effects (font (size 1.27 1.27)) hide)
+    )
+    (property "Field5" "CL21F104ZBCNNNC" (id 8) (at 43.18 66.04 0)
+      (effects (font (size 1.27 1.27)) hide)
+    )
+    (property "Field6" "1276-1007-1-ND" (id 9) (at 43.18 66.04 0)
+      (effects (font (size 1.27 1.27)) hide)
+    )
+    (property "Field7" "C49678" (id 10) (at 43.18 66.04 0)
+      (effects (font (size 1.27 1.27)) hide)
+    )
+    (property "Field8" "CL21F104ZBCNNNC" (id 11) (at 43.18 66.04 0)
+      (effects (font (size 1.27 1.27)) hide)
+    )

Commit message: Bunch of part number updating for JLC
Parts:
- C4: Field4 C49678 -> (none); Field5 CL21F104ZBCNNNC -> (none); Field6 1276-1007-1-ND -> (none); Field7 C49678 -> (none); Field8 CL21F104ZBCNNNC -> (none); LCSC 1276-1007-1-ND -> C14663; MPN C49678 -> CC0603KRX7R9BB104
- SW1: LCSC (none) -> C127509; MPN 1825910-6 -> K2-1102SP-C4SC-04

Commit message: update j6, push buttons back to TH, Part number for j6 was for a 3.81.. (#30)
.. grabbed a random 5mm to use. will probably update pads for buttons yet and maybe different input connector
Parts:
- SW1: LCSC C127509 -> C428628; MPN K2-1102SP-C4SC-04 -> 1825910-6
Changed lines of the file:
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@@
       (effects (font (size 1.27 1.27)) hide)
     )
-    (property "MPN" "K2-1102SP-C4SC-04" (id 5) (at 243.84 46.99 0)
+    (property "MPN" "1825910-6" (id 5) (at 243.84 46.99 0)
       (effects (font (size 1.27 1.27)) hide)
     )
-    (property "LCSC" "C127509" (id 6) (at 243.84 46.99 0)
+    (property "LCSC" "C428628" (id 6) (at 243.84 46.99 0)
       (effects (font (size 1.27 1.27)) hide)
     )
