File: BBB_16_SMD/Diff.kicad_sch (KiCad schematic)
At the start: 7 parts, among them J21 RJ45, U7 AM26C31

Commit message: finished routing
Other:
- title: (none) -> BBB 16 SMD
Changed lines of the file:
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@@
   (paper "A4")
   (title_block
-    (date "2021-11-04")
-    (rev "v2.1")
+    (title "BBB 16 SMD")
+    (date "2022-02-11")
+    (rev "v2")
   )
   (junction (at 153.924 109.22) (diameter 0) (color 0 0 0 0)

Commit message: added boms
Parts:
- C7: Digi-Key_PN 478-7336-1-ND -> 1276-1935-2-ND; LCSC (none) -> C14663; MPN SR215C104KARTR1 -> CL10B104KB8NNWC
- J21: LCSC (none) -> C305972
- R15, R16, R17, R18: Digi-Key_PN 311-120ARCT-ND -> A129677CT-ND; LCSC C17437 -> C22787; MPN RC0805JR-07120RL -> CRGCQ0603F120R
- U7: Digi-Key_PN 296-6785-5-ND -> 296-23457-1-ND; Farnell 4975637 -> (none); LCSC (none) -> C34923; MPN (none) -> AM26C31MDREP
Changed lines of the file:
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@@
       (effects (font (size 1.27 1.27)) hide)
     )
-    (property "Digi-Key_PN" "478-7336-1-ND" (id 5) (at 180.848 101.092 0)
-      (effects (font (size 1.27 1.27)) hide)
-    )
-    (property "MPN" "SR215C104KARTR1" (id 6) (at 180.848 101.092 0)
+    (property "Digi-Key_PN" "1276-1935-2-ND" (id 5) (at 180.848 101.092 0)
+      (effects (font (size 1.27 1.27)) hide)
+    )
+    (property "MPN" "CL10B104KB8NNWC" (id 6) (at 180.848 101.092 0)
+      (effects (font (size 1.27 1.27)) hide)
+    )
+    (property "LCSC" "C14663" (id 7) (at 180.848 101.092 0)
       (effects (font (size 1.27 1.27)) hide)
     )
@@
     )
     (property "MPN" "A-2014-2-4-R" (id 6) (at 78.613 109.093 0)
+      (effects (font (size 1.27 1.27)) hide)
+    )
+    (property "LCSC" "C305972" (id 7) (at 78.613 109.093 0)
       (effects (font (size 1.27 1.27)) hide)
     )
@@
       (effects (font (size 1.27 1.27)) (justify left) hide)
     )
-    (property "Farnell" "4975637" (id 4) (at 150.622 142.24 0)
+    (property "Farnell" "" (id 4) (at 150.622 142.24 0)
       (effects (font (size 1.27 1.27)) (justify left) hide)
     )
@@
       (effects (font (size 1.27 1.27)) hide)
     )
-    (property "Digi-Key_PN" "296-6785-5-ND" (id 6) (at 145.542 116.84 0)
+    (property "Digi-Key_PN" "296-23457-1-ND" (id 6) (at 145.542 116.84 0)
+      (effects (font (size 1.27 1.27)) hide)
+    )
+    (property "LCSC" "C34923" (id 7) (at 145.542 116.84 0)
+      (effects (font (size 1.27 1.27)) hide)
+    )
+    (property "MPN" "AM26C31MDREP" (id 8) (at 145.542 116.84 0)
       (effects (font (size 1.27 1.27)) hide)
     )
@@
       (effects (font (size 1.27 1.27)) hide)
     )
-    (property "Digi-Key_PN" "311-120ARCT-ND" (id 4) (at 102.616 81.661 0)
-      (effects (font (size 1.27 1.27)) hide)
-    )
-    (property "MPN" "RC0805JR-07120RL" (id 5) (at 102.616 81.661 0)
-      (effects (font (size 1.27 1.27)) hide)
-    )
-    (property "LCSC" "C17437" (id 6) (at 102.616 81.661 0)
+    (property "Digi-Key_PN" "A129677CT-ND" (id 4) (at 102.616 81.661 0)
+      (effects (font (size 1.27 1.27)) hide)
+    )
+    (property "MPN" "CRGCQ0603F120R" (id 5) (at 102.616 81.661 0)
+      (effects (font (size 1.27 1.27)) hide)
+    )
+    (property "LCSC" "C22787" (id 6) (at 102.616 81.661 0)
       (effects (font (size 1.27 1.27)) hide)
     )
@@
       (effects (font (size 1.27 1.27)) hide)
     )
-    (property "Digi-Key_PN" "311-120ARCT-ND" (id 4) (at 102.743 76.2 0)
-      (effects (font (size 1.27 1.27)) hide)
-    )
-    (property "MPN" "RC0805JR-07120RL" (id 5) (at 102.743 76.2 0)
-      (effects (font (size 1.27 1.27)) hide)
-    )
-    (property "LCSC" "C17437" (id 6) (at 102.743 76.2 0)
+    (property "Digi-Key_PN" "A129677CT-ND" (id 4) (at 102.743 76.2 0)
+      (effects (font (size 1.27 1.27)) hide)
+    )
+    (property "MPN" "CRGCQ0603F120R" (id 5) (at 102.743 76.2 0)
+      (effects (font (size 1.27 1.27)) hide)
+    )
+    (property "LCSC" "C22787" (id 6) (at 102.743 76.2 0)
       (effects (font (size 1.27 1.27)) hide)
     )
@@
       (effects (font (size 1.27 1.27)) hide)
     )
-    (property "Digi-Key_PN" "311-120ARCT-ND" (id 4) (at 102.87 88.011 0)
-      (effects (font (size 1.27 1.27)) hide)
-    )
-    (property "MPN" "RC0805JR-07120RL" (id 5) (at 102.87 88.011 0)
-      (effects (font (size 1.27 1.27)) hide)
-    )
-    (property "LCSC" "C17437" (id 6) (at 102.87 88.011 0)
+    (property "Digi-Key_PN" "A129677CT-ND" (id 4) (at 102.87 88.011 0)
+      (effects (font (size 1.27 1.27)) hide)
+    )
+    (property "MPN" "CRGCQ0603F120R" (id 5) (at 102.87 88.011 0)
+      (effects (font (size 1.27 1.27)) hide)
+    )
+    (property "LCSC" "C22787" (id 6) (at 102.87 88.011 0)
       (effects (font (size 1.27 1.27)) hide)
     )
@@
       (effects (font (size 1.27 1.27)) hide)
     )
-    (property "Digi-Key_PN" "311-120ARCT-ND" (id 4) (at 102.997 70.993 0)
-      (effects (font (size 1.27 1.27)) hide)
-    )
-    (property "MPN" "RC0805JR-07120RL" (id 5) (at 102.997 70.993 0)
-      (effects (font (size 1.27 1.27)) hide)
-    )
-    (property "LCSC" "C17437" (id 6) (at 102.997 70.993 0)
-      (effects (font (size 1.27 1.27)) hide)
-    )
+    (property "Digi-Key_PN" "A129677CT-ND" (id 4) (at 102.997 70.993 0)
+      (effects (font (size 1.27 1.27)) hide)
+    )
+    (property "MPN" "CRGCQ0603F120R" (id 5) (at 102.997 70.993 0)
+      (effects (font (size 1.27 1.27)) hide)
+    )
+    (property "LCSC" "C22787" (id 6) (at 102.997 70.993 0)
+      (effects (font (size 1.27 1.27)) hide)
+    )

Commit message: Small updates
Update Wrong switch that would force standard pcb vs Economic variant. Update Rj45 PartNumber.
Parts:
- J21: Digi-Key_PN AE10392-ND -> (none); LCSC C305972 -> C2938579; MPN A-2014-2-4-R -> X05ADIWA1DY1022
Changed lines of the file:
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@@
       (effects (font (size 1.27 1.27)) hide)
     )
-    (property "Digi-Key_PN" "AE10392-ND" (id 5) (at 78.613 109.093 0)
+    (property "Digi-Key_PN" "" (id 5) (at 78.613 109.093 0)
       (effects (font (size 1.27 1.27)) hide)
     )
-    (property "MPN" "A-2014-2-4-R" (id 6) (at 78.613 109.093 0)
+    (property "MPN" "X05ADIWA1DY1022" (id 6) (at 78.613 109.093 0)
       (effects (font (size 1.27 1.27)) hide)
     )
-    (property "LCSC" "C305972" (id 7) (at 78.613 109.093 0)
+    (property "LCSC" "C2938579" (id 7) (at 78.613 109.093 0)
       (effects (font (size 1.27 1.27)) hide)
     )

Commit message: reverting bills change
Parts:
- J21: Digi-Key_PN (none) -> AE10392-ND; LCSC C2938579 -> C305972; MPN X05ADIWA1DY1022 -> A-2014-2-4-R
Changed lines of the file:
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@@
       (effects (font (size 1.27 1.27)) hide)
     )
-    (property "Digi-Key_PN" "" (id 5) (at 78.613 109.093 0)
+    (property "Digi-Key_PN" "AE10392-ND" (id 5) (at 78.613 109.093 0)
       (effects (font (size 1.27 1.27)) hide)
     )
-    (property "MPN" "X05ADIWA1DY1022" (id 6) (at 78.613 109.093 0)
+    (property "MPN" "A-2014-2-4-R" (id 6) (at 78.613 109.093 0)
       (effects (font (size 1.27 1.27)) hide)
     )
-    (property "LCSC" "C2938579" (id 7) (at 78.613 109.093 0)
+    (property "LCSC" "C305972" (id 7) (at 78.613 109.093 0)
       (effects (font (size 1.27 1.27)) hide)
     )

Commit message: ~Create some new custom footprints ~Update some JLC PN's ~Updated some 3D model paths
Parts:
- J21: LCSC C305972 -> C2938579; MPN A-2014-2-4-R -> X05ADIWA1DY1022
Changed lines of the file:
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@@
       (effects (font (size 1.27 1.27)) hide)
     )
-    (property "MPN" "A-2014-2-4-R" (id 6) (at 78.613 109.093 0)
+    (property "MPN" "X05ADIWA1DY1022" (id 6) (at 78.613 109.093 0)
       (effects (font (size 1.27 1.27)) hide)
     )
-    (property "LCSC" "C305972" (id 7) (at 78.613 109.093 0)
+    (property "LCSC" "C2938579" (id 7) (at 78.613 109.093 0)
       (effects (font (size 1.27 1.27)) hide)
     )

Commit message: added universal 5V Reg
Other:
- company: (none) -> Scott Hanson
Changed lines of the file:
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@@
   (title_block
     (title "BBB 16 SMD")
-    (date "2022-02-11")
-    (rev "v2")
+    (date "2022-08-14")
+    (rev "v3")
+    (company "Scott Hanson")
   )
   (junction (at 153.924 109.22) (diameter 0) (color 0 0 0 0)
