File: Pi_Zero_W_16_SMD/Serial.kicad_sch (KiCad schematic)
At the start: 14 parts, among them J23 Diff Out, J24 Diff Out, U4 AM26C31, U5 AM26C31

Commit message: added part numbers
Parts:
- C5, C8: Digi-Key_PN (none) -> 1276-1935-2-ND; LCSC (none) -> C14663; MPN (none) -> CL10B104KB8NNWC
- J23, J24: LCSC (none) -> C2938579; MPN A-2014-2-4-R -> X05ADIWA1DY1022
- R10, R11, R12, R13, R14, R7, R8, R9: Digi-Key_PN (none) -> A129677CT-ND; LCSC (none) -> C22787; MPN (none) -> CRGCQ0603F120R
Changed lines of the file:
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@@
       (effects (font (size 1.27 1.27)) hide)
     )
-    (property "MPN" "A-2014-2-4-R" (id 5) (at 27.559 -21.717 0)
+    (property "MPN" "X05ADIWA1DY1022" (id 5) (at 27.559 -21.717 0)
+      (effects (font (size 1.27 1.27)) hide)
+    )
+    (property "LCSC" "C2938579" (id 6) (at 47.625 62.865 0)
       (effects (font (size 1.27 1.27)) hide)
     )
@@
       (effects (font (size 1.27 1.27)) hide)
     )
-    (property "MPN" "A-2014-2-4-R" (id 5) (at 26.924 39.878 0)
+    (property "MPN" "X05ADIWA1DY1022" (id 5) (at 26.924 39.878 0)
+      (effects (font (size 1.27 1.27)) hide)
+    )
+    (property "LCSC" "C2938579" (id 6) (at 49.7078 155.3718 0)
       (effects (font (size 1.27 1.27)) hide)
     )
@@
       (effects (font (size 1.27 1.27)) hide)
     )
-    (property "Digi-Key_PN" "" (id 4) (at 60.96 107.95 0)
-      (effects (font (size 1.27 1.27)) hide)
-    )
-    (property "MPN" "" (id 5) (at 60.96 107.95 0)
-      (effects (font (size 1.27 1.27)) hide)
-    )
-    (property "LCSC" "" (id 6) (at 60.96 107.95 0)
+    (property "Digi-Key_PN" "A129677CT-ND" (id 4) (at 60.96 107.95 0)
+      (effects (font (size 1.27 1.27)) hide)
+    )
+    (property "MPN" "CRGCQ0603F120R" (id 5) (at 60.96 107.95 0)
+      (effects (font (size 1.27 1.27)) hide)
+    )
+    (property "LCSC" "C22787" (id 6) (at 60.96 107.95 0)
       (effects (font (size 1.27 1.27)) hide)
     )
@@
       (effects (font (size 1.27 1.27)) hide)
     )
-    (property "Digi-Key_PN" "" (id 4) (at 60.96 102.87 0)
-      (effects (font (size 1.27 1.27)) hide)
-    )
-    (property "MPN" "" (id 5) (at 60.96 102.87 0)
-      (effects (font (size 1.27 1.27)) hide)
-    )
-    (property "LCSC" "" (id 6) (at 60.96 102.87 0)
+    (property "Digi-Key_PN" "A129677CT-ND" (id 4) (at 60.96 102.87 0)
+      (effects (font (size 1.27 1.27)) hide)
+    )
+    (property "MPN" "CRGCQ0603F120R" (id 5) (at 60.96 102.87 0)
+      (effects (font (size 1.27 1.27)) hide)
+    )
+    (property "LCSC" "C22787" (id 6) (at 60.96 102.87 0)
       (effects (font (size 1.27 1.27)) hide)
     )
@@
       (effects (font (size 1.27 1.27)) hide)
     )
-    (property "Digi-Key_PN" "" (id 4) (at 60.96 120.015 0)
-      (effects (font (size 1.27 1.27)) hide)
-    )
-    (property "MPN" "" (id 5) (at 60.96 120.015 0)
-      (effects (font (size 1.27 1.27)) hide)
-    )
-    (property "LCSC" "" (id 6) (at 60.96 120.015 0)
+    (property "Digi-Key_PN" "A129677CT-ND" (id 4) (at 60.96 120.015 0)
+      (effects (font (size 1.27 1.27)) hide)
+    )
+    (property "MPN" "CRGCQ0603F120R" (id 5) (at 60.96 120.015 0)
+      (effects (font (size 1.27 1.27)) hide)
+    )
+    (property "LCSC" "C22787" (id 6) (at 60.96 120.015 0)
       (effects (font (size 1.27 1.27)) hide)
     )
@@
       (effects (font (size 1.27 1.27)) hide)
     )
-    (property "Digi-Key_PN" "" (id 4) (at 60.96 113.665 0)
-      (effects (font (size 1.27 1.27)) hide)
-    )
-    (property "MPN" "" (id 5) (at 60.96 113.665 0)
-      (effects (font (size 1.27 1.27)) hide)
-    )
-    (property "LCSC" "" (id 6) (at 60.96 113.665 0)
+    (property "Digi-Key_PN" "A129677CT-ND" (id 4) (at 60.96 113.665 0)
+      (effects (font (size 1.27 1.27)) hide)
+    )
+    (property "MPN" "CRGCQ0603F120R" (id 5) (at 60.96 113.665 0)
+      (effects (font (size 1.27 1.27)) hide)
+    )
+    (property "LCSC" "C22787" (id 6) (at 60.96 113.665 0)
       (effects (font (size 1.27 1.27)) hide)
     )
@@
       (effects (font (size 1.27 1.27)) hide)
     )
-    (property "Digi-Key_PN" "" (id 4) (at 124.46 111.125 0)
-      (effects (font (size 1.27 1.27)) hide)
-    )
-    (property "MPN" "" (id 5) (at 124.46 111.125 0)
-      (effects (font (size 1.27 1.27)) hide)
-    )
-    (property "LCSC" "" (id 6) (at 124.46 111.125 0)
+    (property "Digi-Key_PN" "1276-1935-2-ND" (id 4) (at 124.46 111.125 0)
+      (effects (font (size 1.27 1.27)) hide)
+    )
+    (property "MPN" "CL10B104KB8NNWC" (id 5) (at 124.46 111.125 0)
+      (effects (font (size 1.27 1.27)) hide)
+    )
+    (property "LCSC" "C14663" (id 6) (at 124.46 111.125 0)
       (effects (font (size 1.27 1.27)) hide)
     )
@@
       (effects (font (size 1.27 1.27)) hide)
     )
-    (property "Digi-Key_PN" "" (id 4) (at 64.77 59.055 0)
-      (effects (font (size 1.27 1.27)) hide)
-    )
-    (property "MPN" "" (id 5) (at 64.77 59.055 0)
-      (effects (font (size 1.27 1.27)) hide)
-    )
-    (property "LCSC" "" (id 6) (at 64.77 59.055 0)
+    (property "Digi-Key_PN" "A129677CT-ND" (id 4) (at 64.77 59.055 0)
+      (effects (font (size 1.27 1.27)) hide)
+    )
+    (property "MPN" "CRGCQ0603F120R" (id 5) (at 64.77 59.055 0)
+      (effects (font (size 1.27 1.27)) hide)
+    )
+    (property "LCSC" "C22787" (id 6) (at 64.77 59.055 0)
       (effects (font (size 1.27 1.27)) hide)
     )
@@
       (effects (font (size 1.27 1.27)) hide)
     )
-    (property "Digi-Key_PN" "" (id 4) (at 128.27 50.8 0)
-      (effects (font (size 1.27 1.27)) hide)
-    )
-    (property "MPN" "" (id 5) (at 128.27 50.8 0)
-      (effects (font (size 1.27 1.27)) hide)
-    )
-    (property "LCSC" "" (id 6) (at 128.27 50.8 0)
+    (property "Digi-Key_PN" "1276-1935-2-ND" (id 4) (at 128.27 50.8 0)
+      (effects (font (size 1.27 1.27)) hide)
+    )
+    (property "MPN" "CL10B104KB8NNWC" (id 5) (at 128.27 50.8 0)
+      (effects (font (size 1.27 1.27)) hide)
+    )
+    (property "LCSC" "C14663" (id 6) (at 128.27 50.8 0)
       (effects (font (size 1.27 1.27)) hide)
     )
@@
       (effects (font (size 1.27 1.27)) hide)
     )
-    (property "Digi-Key_PN" "" (id 4) (at 64.77 46.99 0)
-      (effects (font (size 1.27 1.27)) hide)
-    )
-    (property "MPN" "" (id 5) (at 64.77 46.99 0)
-      (effects (font (size 1.27 1.27)) hide)
-    )
-    (property "LCSC" "" (id 6) (at 64.77 46.99 0)
+    (property "Digi-Key_PN" "A129677CT-ND" (id 4) (at 64.77 46.99 0)
+      (effects (font (size 1.27 1.27)) hide)
+    )
+    (property "MPN" "CRGCQ0603F120R" (id 5) (at 64.77 46.99 0)
+      (effects (font (size 1.27 1.27)) hide)
+    )
+    (property "LCSC" "C22787" (id 6) (at 64.77 46.99 0)
       (effects (font (size 1.27 1.27)) hide)
     )
@@
       (effects (font (size 1.27 1.27)) hide)
     )
-    (property "Digi-Key_PN" "" (id 4) (at 64.77 41.91 0)
-      (effects (font (size 1.27 1.27)) hide)
-    )
-    (property "MPN" "" (id 5) (at 64.77 41.91 0)
-      (effects (font (size 1.27 1.27)) hide)
-    )
-    (property "LCSC" "" (id 6) (at 64.77 41.91 0)
+    (property "Digi-Key_PN" "A129677CT-ND" (id 4) (at 64.77 41.91 0)
+      (effects (font (size 1.27 1.27)) hide)
+    )
+    (property "MPN" "CRGCQ0603F120R" (id 5) (at 64.77 41.91 0)
+      (effects (font (size 1.27 1.27)) hide)
+    )
+    (property "LCSC" "C22787" (id 6) (at 64.77 41.91 0)
       (effects (font (size 1.27 1.27)) hide)
     )
@@
       (effects (font (size 1.27 1.27)) hide)
     )
-    (property "Digi-Key_PN" "" (id 4) (at 64.135 52.705 0)
-      (effects (font (size 1.27 1.27)) hide)
-    )
-    (property "MPN" "" (id 5) (at 64.135 52.705 0)
-      (effects (font (size 1.27 1.27)) hide)
-    )
-    (property "LCSC" "" (id 6) (at 64.135 52.705 0)
-      (effects (font (size 1.27 1.27)) hide)
-    )
+    (property "Digi-Key_PN" "A129677CT-ND" (id 4) (at 64.135 52.705 0)
+      (effects (font (size 1.27 1.27)) hide)
+    )
+    (property "MPN" "CRGCQ0603F120R" (id 5) (at 64.135 52.705 0)
+      (effects (font (size 1.27 1.27)) hide)
+    )
+    (property "LCSC" "C22787" (id 6) (at 64.135 52.705 0)
+      (effects (font (size 1.27 1.27)) hide)
+    )
