File: Pi_Zero_W_16_SMD/Output9_16.kicad_sch (KiCad schematic)
At the start: 26 parts, among them J10 String10, J11 String11, J12 String12, J13 String13, J14 String14, J15 String15, J16 String16, J9 String9, U3 SN74HCT245N

Commit message: switched to 3.81mm connectors
Parts:
- J10, J11, J12, J13, J14, J15, J16, J9: footprint Connector_Phoenix_MC:PhoenixContact_MCV_1,5_3-G-3.5_1x03_P3.50mm_Vertical -> Scotts:PhoenixContact_MCV_3.81mm_3.5mm_1x03_Vertical
Changed lines of the file:
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@@
       (effects (font (size 1.27 1.27)) (justify left))
     )
-    (property "Footprint" "Connector_Phoenix_MC:PhoenixContact_MCV_1,5_3-G-3.5_1x03_P3.50mm_Vertical" (id 2) (at 149.225 88.265 0)
+    (property "Footprint" "Scotts:PhoenixContact_MCV_3.81mm_3.5mm_1x03_Vertical" (id 2) (at 149.225 88.265 0)
       (effects (font (size 1.27 1.27)) hide)
     )
@@
       (effects (font (size 1.27 1.27)) (justify left))
     )
-    (property "Footprint" "Connector_Phoenix_MC:PhoenixContact_MCV_1,5_3-G-3.5_1x03_P3.50mm_Vertical" (id 2) (at 160.655 88.265 0)
+    (property "Footprint" "Scotts:PhoenixContact_MCV_3.81mm_3.5mm_1x03_Vertical" (id 2) (at 160.655 88.265 0)
       (effects (font (size 1.27 1.27)) hide)
     )
@@
       (effects (font (size 1.27 1.27)) (justify left))
     )
-    (property "Footprint" "Connector_Phoenix_MC:PhoenixContact_MCV_1,5_3-G-3.5_1x03_P3.50mm_Vertical" (id 2) (at 173.355 87.63 0)
+    (property "Footprint" "Scotts:PhoenixContact_MCV_3.81mm_3.5mm_1x03_Vertical" (id 2) (at 173.355 87.63 0)
       (effects (font (size 1.27 1.27)) hide)
     )
@@
       (effects (font (size 1.27 1.27)) (justify left))
     )
-    (property "Footprint" "Connector_Phoenix_MC:PhoenixContact_MCV_1,5_3-G-3.5_1x03_P3.50mm_Vertical" (id 2) (at 186.055 87.63 0)
+    (property "Footprint" "Scotts:PhoenixContact_MCV_3.81mm_3.5mm_1x03_Vertical" (id 2) (at 186.055 87.63 0)
       (effects (font (size 1.27 1.27)) hide)
     )
@@
       (effects (font (size 1.27 1.27)) (justify left))
     )
-    (property "Footprint" "Connector_Phoenix_MC:PhoenixContact_MCV_1,5_3-G-3.5_1x03_P3.50mm_Vertical" (id 2) (at 198.755 86.995 0)
+    (property "Footprint" "Scotts:PhoenixContact_MCV_3.81mm_3.5mm_1x03_Vertical" (id 2) (at 198.755 86.995 0)
       (effects (font (size 1.27 1.27)) hide)
     )
@@
       (effects (font (size 1.27 1.27)) (justify left))
     )
-    (property "Footprint" "Connector_Phoenix_MC:PhoenixContact_MCV_1,5_3-G-3.5_1x03_P3.50mm_Vertical" (id 2) (at 211.455 87.63 0)
+    (property "Footprint" "Scotts:PhoenixContact_MCV_3.81mm_3.5mm_1x03_Vertical" (id 2) (at 211.455 87.63 0)
       (effects (font (size 1.27 1.27)) hide)
     )
@@
       (effects (font (size 1.27 1.27)) (justify left))
     )
-    (property "Footprint" "Connector_Phoenix_MC:PhoenixContact_MCV_1,5_3-G-3.5_1x03_P3.50mm_Vertical" (id 2) (at 224.79 86.995 0)
+    (property "Footprint" "Scotts:PhoenixContact_MCV_3.81mm_3.5mm_1x03_Vertical" (id 2) (at 224.79 86.995 0)
       (effects (font (size 1.27 1.27)) hide)
     )
@@
       (effects (font (size 1.27 1.27)) (justify left))
     )
-    (property "Footprint" "Connector_Phoenix_MC:PhoenixContact_MCV_1,5_3-G-3.5_1x03_P3.50mm_Vertical" (id 2) (at 237.49 86.995 0)
+    (property "Footprint" "Scotts:PhoenixContact_MCV_3.81mm_3.5mm_1x03_Vertical" (id 2) (at 237.49 86.995 0)
       (effects (font (size 1.27 1.27)) hide)
     )

Commit message: added part numbers
Parts:
- C4: Digi-Key_PN (none) -> 1276-1935-2-ND; LCSC (none) -> C14663; MPN (none) -> CL10B104KB8NNWC
- F10, F11, F12, F13, F14, F15, F16, F9: LCSC (none) -> C492610
- J10, J11, J12, J13, J14, J15, J16, J9: LCSC (none) -> C192778
- R23, R24, R25, R26, R27, R28, R29, R30: Digi-Key_PN (none) -> 311-33.0HRCT-ND; LCSC (none) -> C23140; MPN (none) -> RC0603FR-0733RL
Changed lines of the file:
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@@
+      (effects (font (size 1.27 1.27)) hide)
+    )
+    (property "LCSC" "C192778" (id 6) (at 147.701 83.693 0)
       (effects (font (size 1.27 1.27)) hide)
     )
@@
       (effects (font (size 1.27 1.27)) hide)
     )
+    (property "LCSC" "C192778" (id 6) (at 159.131 83.439 0)
+      (effects (font (size 1.27 1.27)) hide)
+    )
     (pin "1")
     (pin "2")
@@
       (effects (font (size 1.27 1.27)) hide)
     )
+    (property "LCSC" "C192778" (id 6) (at 171.831 82.804 0)
+      (effects (font (size 1.27 1.27)) hide)
+    )
     (pin "1")
     (pin "2")
@@
       (effects (font (size 1.27 1.27)) hide)
     )
+    (property "LCSC" "C192778" (id 6) (at 185.039 82.804 0)
+      (effects (font (size 1.27 1.27)) hide)
+    )
     (pin "1")
     (pin "2")
@@
       (effects (font (size 1.27 1.27)) hide)
     )
+    (property "LCSC" "C192778" (id 6) (at 197.231 82.169 0)
+      (effects (font (size 1.27 1.27)) hide)
+    )
     (pin "1")
     (pin "2")
@@
       (effects (font (size 1.27 1.27)) hide)
     )
+    (property "LCSC" "C192778" (id 6) (at 209.931 82.55 0)
+      (effects (font (size 1.27 1.27)) hide)
+    )
     (pin "1")
     (pin "2")
@@
       (effects (font (size 1.27 1.27)) hide)
     )
+    (property "LCSC" "C192778" (id 6) (at 223.52 82.169 0)
+      (effects (font (size 1.27 1.27)) hide)
+    )
     (pin "1")
     (pin "2")
@@
     )
     (property "MPN" "1843619/OSTTJ0311530" (id 5) (at -19.812 -16.383 0)
+      (effects (font (size 1.27 1.27)) hide)
+    )
+    (property "LCSC" "C192778" (id 6) (at 236.22 82.169 0)
       (effects (font (size 1.27 1.27)) hide)
     )
@@
     )
     (property "MPN" "3544-2" (id 10) (at 73.152 -133.985 0)
+      (effects (font (size 1.27 1.27)) hide)
+    )
+    (property "LCSC" "C492610" (id 11) (at 159.512 65.5066 0)
       (effects (font (size 1.27 1.27)) hide)
     )
@@
       (effects (font (size 1.27 1.27)) hide)
     )
+    (property "LCSC" "C492610" (id 11) (at 171.577 66.1416 0)
+      (effects (font (size 1.27 1.27)) hide)
+    )
     (pin "1_1")
     (pin "1_2")
@@
       (effects (font (size 1.27 1.27)) hide)
     )
+    (property "LCSC" "C492610" (id 11) (at 184.277 66.1416 0)
+      (effects (font (size 1.27 1.27)) hide)
+    )
     (pin "1_1")
     (pin "1_2")
@@
       (effects (font (size 1.27 1.27)) hide)
     )
+    (property "LCSC" "C492610" (id 11) (at 196.977 66.1416 0)
+      (effects (font (size 1.27 1.27)) hide)
+    )
     (pin "1_1")
     (pin "1_2")
@@
       (effects (font (size 1.27 1.27)) hide)
     )
+    (property "LCSC" "C492610" (id 11) (at 209.677 65.5066 0)
+      (effects (font (size 1.27 1.27)) hide)
+    )
     (pin "1_1")
     (pin "1_2")
@@
       (effects (font (size 1.27 1.27)) hide)
     )
+    (property "LCSC" "C492610" (id 11) (at 223.012 65.5066 0)
+      (effects (font (size 1.27 1.27)) hide)
+    )
     (pin "1_1")
     (pin "1_2")
@@
       (effects (font (size 1.27 1.27)) hide)
     )
+    (property "LCSC" "C492610" (id 11) (at 235.712 65.5066 0)
+      (effects (font (size 1.27 1.27)) hide)
+    )
     (pin "1_1")
     (pin "1_2")
@@
       (effects (font (size 1.27 1.27)) hide)
     )
-    (property "Digi-Key_PN" "" (id 4) (at 132.715 93.98 0)
-      (effects (font (size 1.27 1.27)) hide)
-    )
-    (property "MPN" "" (id 5) (at 132.715 93.98 0)
-      (effects (font (size 1.27 1.27)) hide)
-    )
-    (property "LCSC" "" (id 6) (at 132.715 93.98 0)
+    (property "Digi-Key_PN" "1276-1935-2-ND" (id 4) (at 132.715 93.98 0)
+      (effects (font (size 1.27 1.27)) hide)
+    )
+    (property "MPN" "CL10B104KB8NNWC" (id 5) (at 132.715 93.98 0)
+      (effects (font (size 1.27 1.27)) hide)
+    )
+    (property "LCSC" "C14663" (id 6) (at 132.715 93.98 0)
       (effects (font (size 1.27 1.27)) hide)
     )
@@
       (effects (font (size 1.27 1.27)) hide)
     )
+    (property "LCSC" "C492610" (id 11) (at 147.447 66.1416 0)
+      (effects (font (size 1.27 1.27)) hide)
+    )
     (pin "1_1")
     (pin "1_2")
@@
       (effects (font (size 1.27 1.27)) hide)
     )
-    (property "LCSC" "" (id 4) (at 132.715 115.57 0)
-      (effects (font (size 1.27 1.27)) hide)
-    )
-    (property "Digi-Key_PN" "" (id 5) (at 132.715 115.57 0)
-      (effects (font (size 1.27 1.27)) hide)
-    )
-    (property "MPN" "" (id 6) (at 132.715 115.57 0)
+    (property "LCSC" "C23140" (id 4) (at 132.715 115.57 0)
+      (effects (font (size 1.27 1.27)) hide)
+    )
+    (property "Digi-Key_PN" "311-33.0HRCT-ND" (id 5) (at 132.715 115.57 0)
+      (effects (font (size 1.27 1.27)) hide)
+    )
+    (property "MPN" "RC0603FR-0733RL" (id 6) (at 132.715 115.57 0)
       (effects (font (size 1.27 1.27)) hide)
     )
@@
       (effects (font (size 1.27 1.27)) hide)
     )
-    (property "LCSC" "" (id 4) (at 132.715 113.03 0)
-      (effects (font (size 1.27 1.27)) hide)
-    )
-    (property "Digi-Key_PN" "" (id 5) (at 132.715 113.03 0)
-      (effects (font (size 1.27 1.27)) hide)
-    )
-    (property "MPN" "" (id 6) (at 132.715 113.03 0)
+    (property "LCSC" "C23140" (id 4) (at 132.715 113.03 0)
+      (effects (font (size 1.27 1.27)) hide)
+    )
+    (property "Digi-Key_PN" "311-33.0HRCT-ND" (id 5) (at 132.715 113.03 0)
+      (effects (font (size 1.27 1.27)) hide)
+    )
+    (property "MPN" "RC0603FR-0733RL" (id 6) (at 132.715 113.03 0)
       (effects (font (size 1.27 1.27)) hide)
     )
@@
       (effects (font (size 1.27 1.27)) hide)
     )
-    (property "LCSC" "" (id 4) (at 132.715 118.11 0)
-      (effects (font (size 1.27 1.27)) hide)
-    )
-    (property "Digi-Key_PN" "" (id 5) (at 132.715 118.11 0)
-      (effects (font (size 1.27 1.27)) hide)
-    )
-    (property "MPN" "" (id 6) (at 132.715 118.11 0)
+    (property "LCSC" "C23140" (id 4) (at 132.715 118.11 0)
+      (effects (font (size 1.27 1.27)) hide)
+    )
+    (property "Digi-Key_PN" "311-33.0HRCT-ND" (id 5) (at 132.715 118.11 0)
+      (effects (font (size 1.27 1.27)) hide)
+    )
+    (property "MPN" "RC0603FR-0733RL" (id 6) (at 132.715 118.11 0)
       (effects (font (size 1.27 1.27)) hide)
     )
@@
       (effects (font (size 1.27 1.27)) hide)
     )
-    (property "LCSC" "" (id 4) (at 132.715 110.49 0)
-      (effects (font (size 1.27 1.27)) hide)
-    )
-    (property "Digi-Key_PN" "" (id 5) (at 132.715 110.49 0)
-      (effects (font (size 1.27 1.27)) hide)
-    )
-    (property "MPN" "" (id 6) (at 132.715 110.49 0)
+    (property "LCSC" "C23140" (id 4) (at 132.715 110.49 0)
+      (effects (font (size 1.27 1.27)) hide)
+    )
+    (property "Digi-Key_PN" "311-33.0HRCT-ND" (id 5) (at 132.715 110.49 0)
+      (effects (font (size 1.27 1.27)) hide)
+    )
+    (property "MPN" "RC0603FR-0733RL" (id 6) (at 132.715 110.49 0)
       (effects (font (size 1.27 1.27)) hide)
     )
@@
       (effects (font (size 1.27 1.27)) hide)
     )
-    (property "LCSC" "" (id 4) (at 132.715 100.33 0)
-      (effects (font (size 1.27 1.27)) hide)
-    )
-    (property "Digi-Key_PN" "" (id 5) (at 132.715 100.33 0)
-      (effects (font (size 1.27 1.27)) hide)
-    )
-    (property "MPN" "" (id 6) (at 132.715 100.33 0)
+    (property "LCSC" "C23140" (id 4) (at 132.715 100.33 0)
+      (effects (font (size 1.27 1.27)) hide)
+    )
+    (property "Digi-Key_PN" "311-33.0HRCT-ND" (id 5) (at 132.715 100.33 0)
+      (effects (font (size 1.27 1.27)) hide)
+    )
+    (property "MPN" "RC0603FR-0733RL" (id 6) (at 132.715 100.33 0)
       (effects (font (size 1.27 1.27)) hide)
     )
@@
       (effects (font (size 1.27 1.27)) hide)
     )
-    (property "LCSC" "" (id 4) (at 132.715 107.95 0)
-      (effects (font (size 1.27 1.27)) hide)
-    )
-    (property "Digi-Key_PN" "" (id 5) (at 132.715 107.95 0)
-      (effects (font (size 1.27 1.27)) hide)
-    )
-    (property "MPN" "" (id 6) (at 132.715 107.95 0)
+    (property "LCSC" "C23140" (id 4) (at 132.715 107.95 0)
+      (effects (font (size 1.27 1.27)) hide)
+    )
+    (property "Digi-Key_PN" "311-33.0HRCT-ND" (id 5) (at 132.715 107.95 0)
+      (effects (font (size 1.27 1.27)) hide)
+    )
+    (property "MPN" "RC0603FR-0733RL" (id 6) (at 132.715 107.95 0)
       (effects (font (size 1.27 1.27)) hide)
     )
@@
       (effects (font (size 1.27 1.27)) hide)
     )
-    (property "LCSC" "" (id 4) (at 132.715 105.41 0)
-      (effects (font (size 1.27 1.27)) hide)
-    )
-    (property "Digi-Key_PN" "" (id 5) (at 132.715 105.41 0)
-      (effects (font (size 1.27 1.27)) hide)
-    )
-    (property "MPN" "" (id 6) (at 132.715 105.41 0)
+    (property "LCSC" "C23140" (id 4) (at 132.715 105.41 0)
+      (effects (font (size 1.27 1.27)) hide)
+    )
+    (property "Digi-Key_PN" "311-33.0HRCT-ND" (id 5) (at 132.715 105.41 0)
+      (effects (font (size 1.27 1.27)) hide)
+    )
+    (property "MPN" "RC0603FR-0733RL" (id 6) (at 132.715 105.41 0)
       (effects (font (size 1.27 1.27)) hide)
     )
@@
       (effects (font (size 1.27 1.27)) hide)
     )
-    (property "LCSC" "" (id 4) (at 132.715 102.87 0)
-      (effects (font (size 1.27 1.27)) hide)
-    )
-    (property "Digi-Key_PN" "" (id 5) (at 132.715 102.87 0)
-      (effects (font (size 1.27 1.27)) hide)
-    )
-    (property "MPN" "" (id 6) (at 132.715 102.87 0)
-      (effects (font (size 1.27 1.27)) hide)
-    )
+    (property "LCSC" "C23140" (id 4) (at 132.715 102.87 0)
+      (effects (font (size 1.27 1.27)) hide)
+    )
+    (property "Digi-Key_PN" "311-33.0HRCT-ND" (id 5) (at 132.715 102.87 0)
+      (effects (font (size 1.27 1.27)) hide)
+    )
+    (property "MPN" "RC0603FR-0733RL" (id 6) (at 132.715 102.87 0)
+      (effects (font (size 1.27 1.27)) hide)
+    )

Commit message: update
Parts:
- J10, J11, J12, J13, J14, J15, J16, J9: LCSC C192778 -> C8389
Changed lines of the file:
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@@
       (effects (font (size 1.27 1.27)) hide)
     )
-    (property "LCSC" "C192778" (id 6) (at 147.701 83.693 0)
+    (property "LCSC" "C8389" (id 6) (at 147.701 83.693 0)
       (effects (font (size 1.27 1.27)) hide)
     )
@@
       (effects (font (size 1.27 1.27)) hide)
     )
-    (property "LCSC" "C192778" (id 6) (at 159.131 83.439 0)
+    (property "LCSC" "C8389" (id 6) (at 159.131 83.439 0)
       (effects (font (size 1.27 1.27)) hide)
     )
@@
       (effects (font (size 1.27 1.27)) hide)
     )
-    (property "LCSC" "C192778" (id 6) (at 171.831 82.804 0)
+    (property "LCSC" "C8389" (id 6) (at 171.831 82.804 0)
       (effects (font (size 1.27 1.27)) hide)
     )
@@
       (effects (font (size 1.27 1.27)) hide)
     )
-    (property "LCSC" "C192778" (id 6) (at 185.039 82.804 0)
+    (property "LCSC" "C8389" (id 6) (at 185.039 82.804 0)
       (effects (font (size 1.27 1.27)) hide)
     )
@@
       (effects (font (size 1.27 1.27)) hide)
     )
-    (property "LCSC" "C192778" (id 6) (at 197.231 82.169 0)
+    (property "LCSC" "C8389" (id 6) (at 197.231 82.169 0)
       (effects (font (size 1.27 1.27)) hide)
     )
@@
       (effects (font (size 1.27 1.27)) hide)
     )
-    (property "LCSC" "C192778" (id 6) (at 209.931 82.55 0)
+    (property "LCSC" "C8389" (id 6) (at 209.931 82.55 0)
       (effects (font (size 1.27 1.27)) hide)
     )
@@
       (effects (font (size 1.27 1.27)) hide)
     )
-    (property "LCSC" "C192778" (id 6) (at 223.52 82.169 0)
+    (property "LCSC" "C8389" (id 6) (at 223.52 82.169 0)
       (effects (font (size 1.27 1.27)) hide)
     )
@@
       (effects (font (size 1.27 1.27)) hide)
     )
-    (property "LCSC" "C192778" (id 6) (at 236.22 82.169 0)
+    (property "LCSC" "C8389" (id 6) (at 236.22 82.169 0)
       (effects (font (size 1.27 1.27)) hide)
     )
