File: Pi_CM4_16_SMD/Output1_8.kicad_sch (KiCad schematic)
At the start: 26 parts, among them J11 String8, J12 String1, J13 String2, J14 String3, J15 String4, J16 String5, J17 String6, J18 String7, U8 SN74HCT245N

Commit message: removed rescue library
Parts:
- U8: symbol Pi_CM4_16-rescue:SN74HCT245N-SN74HCT245N -> Scotts:SN74HCT245N
Changed lines of the file:
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@@
     (pin "1")
   )
-  (symbol (lib_id "Pi_CM4_16-rescue:SN74HCT245N-SN74HCT245N") (at 76.835 94.615 0) (unit 1)
+  (symbol (lib_id "Scotts:SN74HCT245N") (at 76.835 94.615 0) (unit 1)
     (in_bom yes) (on_board yes)
     (property "Reference" "U8" (id 0) (at 104.267 85.979 0)
