File: Teensy_16_SMD/Teensy_16.kicad_sch (KiCad schematic)
At the start: 34 parts, among them J17 Power In Left, J18 Power In Right, J19 GPIO, J23 VIN Voltage, J24 Expansion Header, J26 OLED, J27 Aux Pwr, J28 VIN Select, Q1 DMP3056L, U2 AMS1117-5.0

Commit message: added PCB for walmart tree
Parts:
- PIN3: value (none) -> Jumper; footprint (none) -> Jumper:SolderJumper-3_P1.3mm_Bridged12_Pad1.0x1.5mm
- PIN4: value (none) -> JUMPER; footprint (none) -> Jumper:SolderJumper-3_P1.3mm_Bridged12_Pad1.0x1.5mm
Changed lines of the file:
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@@
     (in_bom yes) (on_board yes)
     (property "Reference" "PIN3" (id 0) (at 52.578 31.75 0))
-    (property "Value" "" (id 1) (at 52.324 31.9024 0)
+    (property "Value" "Jumper" (id 1) (at 52.324 31.9024 0)
       (effects (font (size 1.27 1.27)) hide)
     )
-    (property "Footprint" "" (id 2) (at 52.324 34.798 0)
+    (property "Footprint" "Jumper:SolderJumper-3_P1.3mm_Bridged12_Pad1.0x1.5mm" (id 2) (at 52.324 34.798 0)
       (effects (font (size 1.27 1.27)) hide)
     )
@@
     (in_bom yes) (on_board yes)
     (property "Reference" "PIN4" (id 0) (at 41.529 47.8282 0))
-    (property "Value" "" (id 1) (at 41.529 50.1396 0)
+    (property "Value" "JUMPER" (id 1) (at 41.529 50.1396 0)
       (effects (font (size 1.27 1.27)) hide)
     )
-    (property "Footprint" "" (id 2) (at 41.529 44.958 0)
+    (property "Footprint" "Jumper:SolderJumper-3_P1.3mm_Bridged12_Pad1.0x1.5mm" (id 2) (at 41.529 44.958 0)
       (effects (font (size 1.27 1.27)) hide)
     )
