File: Pi_Zero_W_2_SMD/Pi_Zero_W_2.kicad_sch (KiCad schematic)
At the start: 26 parts, among them J3 Power In Right, J5 VIN Voltage, J6 OLED Conn, Q1 DMP3056L, SW1 Down BTN, SW2 Enter BTN, U1 Universe5V, U2 24LC256

Commit message: updates
Parts:
- J3: Digi-Key_PN ED2953-ND -> (none); LCSC C707421 -> C306200; MPN OSTYK51102030 -> (none)
Other:
- title: Pi_Zero_W_2 -> Pi Zero W 2
Changed lines of the file:
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@@
 	(paper "A4")
 	(title_block
-		(title "Pi_Zero_W_2")
-		(date "2022-08-20")
+		(title "Pi Zero W 2")
+		(date "2024-12-30")
 		(rev "v1")
 		(company "Scott Hanson")
@@
 			)
 		)
-		(property "Digi-Key_PN" "ED2953-ND"
+		(property "Digi-Key_PN" ""
 			(at 38.735 46.99 0)
 			(effects
@@
 			)
 		)
-		(property "MPN" "OSTYK51102030"
+		(property "MPN" ""
 			(at 38.735 46.99 0)
 			(effects
@@
 			)
 		)
-		(property "LCSC" "C707421"
+		(property "LCSC" "C306200"
 			(at 40.8178 41.4782 0)
 			(effects
