File: Receiver_Out_Edge_SMD/Receiver_Out.kicad_sch (KiCad schematic)
At the start: 23 parts, among them J5 PGM, J6 VIN_Voltage, J8 Conn_ARM_SWD_TagConnect_TC203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, J9 XT60PW-M, SW1 Test, U2 AMS1117-5.0, U5 ATtiny1616-M

Commit message: more work on edge version
Parts:
- removed H1, H2, H3, H4: MountingHole, Scotts:MountingHole_3.7mm, symbol Mechanical:MountingHole
- added JP1: Vin_Jumper, Jumper:SolderJumper-3_P2.0mm_Open_TrianglePad1.0x1.5mm, symbol Jumper:SolderJumper_3_Open
Connections:
- net +5V: now also JP1.3 (B)
- net PWR: now also JP1.1 (A)
- net VIN: now also JP1.2 (C)
Other:
- title: Receiver Out SMD -> Receiver Out Edge
- moved on the sheet: C1, C2, C5, D1, D2, D3, D4, D5, J5, J6, J8, J9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
