File: Receiver_Out_Edge_SMD/Diff_In.kicad_sch (KiCad schematic)
At the start: 8 parts, among them J7 RJ45, U3 AM26C32IN

Commit message: more work on edge version
Other:
- title: Receiver Out SMD -> Receiver Out Edge
Changed lines of the file:
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@@
 	(paper "A4")
 	(title_block
-		(title "Receiver Out SMD")
-		(date "2025-02-23")
-		(rev "v3")
+		(title "Receiver Out Edge")
+		(date "2026-02-22")
+		(rev "v1")
 		(company "Scott Hanson")
 	)

Commit message: fixes
Parts:
- R?: renamed from R12; now fitted; now in the parts list
- renumbered C4 to C?, J7 to J?, R3 to R?, R4 to R?, R5 to R?, R6 to R?, U3 to U?
Changed lines of the file:
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@@
 		(on_board yes)
 		(dnp no)
-		(property "Reference" "U3"
+		(property "Reference" "U?"
 			(at 135.128 97.028 0)
 			(effects
@@
 		)
 		(instances
+			(project "Diff_In"
+				(path "/454df662-9f7f-45dc-9fbe-e6ec06511907"
+					(reference "U?")
+					(unit 1)
+				)
+			)
 			(project "Receiver_Out"
 				(path "/95254009-634e-4d56-880f-446c022a099c/00000000-0000-0000-0000-00005e06688b"
@@
 		(on_board yes)
 		(dnp no)
-		(property "Reference" "J7"
+		(property "Reference" "J?"
 			(at 150.622 67.5894 90)
 			(effects
@@
 		)
 		(instances
+			(project "Diff_In"
+				(path "/454df662-9f7f-45dc-9fbe-e6ec06511907"
+					(reference "J?")
+					(unit 1)
+				)
+			)
 			(project "Receiver_Out"
 				(path "/95254009-634e-4d56-880f-446c022a099c/00000000-0000-0000-0000-00005e06688b"
@@
 		(on_board yes)
 		(dnp no)
-		(property "Reference" "#PWR017"
+		(property "Reference" "#PWR?"
 			(at 156.21 106.68 0)
 			(effects
@@
 		)
 		(instances
+			(project "Diff_In"
+				(path "/454df662-9f7f-45dc-9fbe-e6ec06511907"
+					(reference "#PWR?")
+					(unit 1)
+				)
+			)
 			(project "Receiver_Out"
 				(path "/95254009-634e-4d56-880f-446c022a099c/00000000-0000-0000-0000-00005e06688b"
@@
 		(on_board yes)
 		(dnp no)
-		(property "Reference" "#PWR018"
+		(property "Reference" "#PWR?"
 			(at 90.17 124.46 0)
 			(effects
@@
 		)
 		(instances
+			(project "Diff_In"
+				(path "/454df662-9f7f-45dc-9fbe-e6ec06511907"
+					(reference "#PWR?")
+					(unit 1)
+				)
+			)
 			(project "Receiver_Out"
 				(path "/95254009-634e-4d56-880f-446c022a099c/00000000-0000-0000-0000-00005e06688b"
@@
 		(on_board yes)
 		(dnp no)
-		(property "Reference" "#PWR016"
+		(property "Reference" "#PWR?"
 			(at 110.49 129.54 0)
 			(effects
@@
 		)
 		(instances
+			(project "Diff_In"
+				(path "/454df662-9f7f-45dc-9fbe-e6ec06511907"
+					(reference "#PWR?")
+					(unit 1)
+				)
+			)
 			(project "Receiver_Out"
 				(path "/95254009-634e-4d56-880f-446c022a099c/00000000-0000-0000-0000-00005e06688b"
@@
 		(on_board yes)
 		(dnp no)
-		(property "Reference" "C4"
+		(property "Reference" "C?"
 			(at 195.961 95.3516 0)
 			(effects
@@
 		)
 		(instances
+			(project "Diff_In"
+				(path "/454df662-9f7f-45dc-9fbe-e6ec06511907"
+					(reference "C?")
+					(unit 1)
+				)
+			)
 			(project "Receiver_Out"
 				(path "/95254009-634e-4d56-880f-446c022a099c/00000000-0000-0000-0000-00005e06688b"
@@
 		(on_board yes)
 		(dnp no)
-		(property "Reference" "#PWR024"
+		(property "Reference" "#PWR?"
 			(at 193.04 106.68 0)
 			(effects
@@
 		)
 		(instances
+			(project "Diff_In"
+				(path "/454df662-9f7f-45dc-9fbe-e6ec06511907"
+					(reference "#PWR?")
+					(unit 1)
+				)
+			)
 			(project "Receiver_Out"
 				(path "/95254009-634e-4d56-880f-446c022a099c/00000000-0000-0000-0000-00005e06688b"
@@
 		(on_board yes)
 		(dnp no)
-		(property "Reference" "#PWR023"
+		(property "Reference" "#PWR?"
 			(at 193.04 96.52 0)
 			(effects
@@
 		)
 		(instances
+			(project "Diff_In"
+				(path "/454df662-9f7f-45dc-9fbe-e6ec06511907"
+					(reference "#PWR?")
+					(unit 1)
+				)
+			)
 			(project "Receiver_Out"
 				(path "/95254009-634e-4d56-880f-446c022a099c/00000000-0000-0000-0000-00005e06688b"
@@
 		(on_board yes)
 		(dnp no)
-		(property "Reference" "R3"
+		(property "Reference" "R?"
 			(at 99.06 98.8822 90)
 			(effects
@@
 		)
 		(instances
+			(project "Diff_In"
+				(path "/454df662-9f7f-45dc-9fbe-e6ec06511907"
+					(reference "R?")
+					(unit 1)
+				)
+			)
 			(project "Receiver_Out"
 				(path "/95254009-634e-4d56-880f-446c022a099c/00000000-0000-0000-0000-00005e06688b"
@@
 		(on_board yes)
 		(dnp no)
-		(property "Reference" "R4"
+		(property "Reference" "R?"
 			(at 109.22 97.6122 90)
 			(effects
@@
 		)
 		(instances
+			(project "Diff_In"
+				(path "/454df662-9f7f-45dc-9fbe-e6ec06511907"
+					(reference "R?")
+					(unit 1)
+				)
+			)
 			(project "Receiver_Out"
 				(path "/95254009-634e-4d56-880f-446c022a099c/00000000-0000-0000-0000-00005e06688b"
@@
 		(on_board yes)
 		(dnp no)
-		(property "Reference" "R5"
+		(property "Reference" "R?"
 			(at 163.83 98.8822 90)
 			(effects
@@
 		)
 		(instances
+			(project "Diff_In"
+				(path "/454df662-9f7f-45dc-9fbe-e6ec06511907"
+					(reference "R?")
+					(unit 1)
+				)
+			)
 			(project "Receiver_Out"
 				(path "/95254009-634e-4d56-880f-446c022a099c/00000000-0000-0000-0000-00005e06688b"
@@
 		(on_board yes)
 		(dnp no)
-		(property "Reference" "R6"
+		(property "Reference" "R?"
 			(at 180.34 100.1522 90)
 			(effects
@@
 		)
 		(instances
+			(project "Diff_In"
+				(path "/454df662-9f7f-45dc-9fbe-e6ec06511907"
+					(reference "R?")
+					(unit 1)
+				)
+			)
 			(project "Receiver_Out"
 				(path "/95254009-634e-4d56-880f-446c022a099c/00000000-0000-0000-0000-00005e06688b"
@@
 		(unit 1)
 		(exclude_from_sim no)
-		(in_bom no)
-		(on_board yes)
-		(dnp yes)
-		(property "Reference" "R12"
+		(in_bom yes)
+		(on_board yes)
+		(dnp no)
+		(property "Reference" "R?"
 			(at 159.8422 128.27 90)
 			(effects
@@
 		)
 		(instances
+			(project "Diff_In"
+				(path "/454df662-9f7f-45dc-9fbe-e6ec06511907"
+					(reference "R?")
+					(unit 1)
+				)
+			)
 			(project "Receiver_Out"
 				(path "/95254009-634e-4d56-880f-446c022a099c/00000000-0000-0000-0000-00005e06688b"
@@
 		(on_board yes)
 		(dnp no)
-		(property "Reference" "#PWR027"
+		(property "Reference" "#PWR?"
 			(at 165.1 140.97 0)
 			(effects
@@
 		)
 		(instances
+			(project "Diff_In"
+				(path "/454df662-9f7f-45dc-9fbe-e6ec06511907"
+					(reference "#PWR?")
+					(unit 1)
+				)
+			)
 			(project "Receiver_Out"
 				(path "/95254009-634e-4d56-880f-446c022a099c/00000000-0000-0000-0000-00005e06688b"
@@
 		)
 	)
+	(sheet_instances
+		(path "/"
+			(page "1")
+		)
+	)
+	(embedded_fonts no)
 )
