File: BBB_16/Output1_8.kicad_sch (KiCad schematic)
At the start: 20 parts, among them J1 String1, J2 String2, J3 String3, J4 String4, J5 String5, J6 String6, J7 String7, J8 String8, U3 SN74HCT245N

Commit message: added cut trace to OLED power pins
Parts:
- F1, F2, F3, F4, F5, F6, F7, F8: footprint Keystone_Fuse:FUSE_3544-2 -> Scotts:FUSE_3544-2
Changed lines of the file:
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@@
   (title_block
     (title "BBB 16")
-    (date "2022-08-14")
-    (rev "v2.2")
+    (date "2023-02-02")
+    (rev "v2.3")
     (company "Scott Hanson")
   )
@@
       (effects (font (size 1.27 1.27)) (justify left))
     )
-    (property "Footprint" "Keystone_Fuse:FUSE_3544-2" (id 2) (at 157.226 80.772 0)
+    (property "Footprint" "Scotts:FUSE_3544-2" (id 2) (at 157.226 80.772 0)
       (effects (font (size 1.27 1.27)) (justify left bottom) hide)
     )
@@
       (effects (font (size 1.27 1.27)) (justify left))
     )
-    (property "Footprint" "Keystone_Fuse:FUSE_3544-2" (id 2) (at 168.91 81.026 0)
+    (property "Footprint" "Scotts:FUSE_3544-2" (id 2) (at 168.91 81.026 0)
       (effects (font (size 1.27 1.27)) (justify left bottom) hide)
     )
@@
       (effects (font (size 1.27 1.27)) (justify left))
     )
-    (property "Footprint" "Keystone_Fuse:FUSE_3544-2" (id 2) (at 180.34 81.28 0)
+    (property "Footprint" "Scotts:FUSE_3544-2" (id 2) (at 180.34 81.28 0)
       (effects (font (size 1.27 1.27)) (justify left bottom) hide)
     )
@@
       (effects (font (size 1.27 1.27)) (justify left))
     )
-    (property "Footprint" "Keystone_Fuse:FUSE_3544-2" (id 2) (at 191.77 81.026 0)
+    (property "Footprint" "Scotts:FUSE_3544-2" (id 2) (at 191.77 81.026 0)
       (effects (font (size 1.27 1.27)) (justify left bottom) hide)
     )
@@
       (effects (font (size 1.27 1.27)) (justify left))
     )
-    (property "Footprint" "Keystone_Fuse:FUSE_3544-2" (id 2) (at 203.2 80.772 0)
+    (property "Footprint" "Scotts:FUSE_3544-2" (id 2) (at 203.2 80.772 0)
       (effects (font (size 1.27 1.27)) (justify left bottom) hide)
     )
@@
       (effects (font (size 1.27 1.27)) (justify left))
     )
-    (property "Footprint" "Keystone_Fuse:FUSE_3544-2" (id 2) (at 214.63 80.772 0)
+    (property "Footprint" "Scotts:FUSE_3544-2" (id 2) (at 214.63 80.772 0)
       (effects (font (size 1.27 1.27)) (justify left bottom) hide)
     )
@@
       (effects (font (size 1.27 1.27)) (justify left))
     )
-    (property "Footprint" "Keystone_Fuse:FUSE_3544-2" (id 2) (at 226.06 80.772 0)
+    (property "Footprint" "Scotts:FUSE_3544-2" (id 2) (at 226.06 80.772 0)
       (effects (font (size 1.27 1.27)) (justify left bottom) hide)
     )
@@
       (effects (font (size 1.27 1.27)) (justify left))
     )
-    (property "Footprint" "Keystone_Fuse:FUSE_3544-2" (id 2) (at 145.796 81.026 0)
-      (effects (font (size 1.27 1.27)) (justify left bottom) hide)
-    )
+    (property "Footprint" "Scotts:FUSE_3544-2" (id 2) (at 145.796 81.026 0)
+      (effects (font (size 1.27 1.27)) (justify left bottom) hide)
+    )
