File: Four_Out/Four_Out.kicad_sch (KiCad schematic)
At the start: 9 parts

Commit message: updates
Parts:
- added H1, H2, H3, H4: MountingHole, Scotts:MountingHole_3.7mm, symbol Mechanical:MountingHole
- D1: value (none) -> SB5100-T; footprint (none) -> Diode_THT:D_DO-201AD_P12.70mm_Horizontal
- D2: value (none) -> VIN LED; footprint (none) -> LED_THT:LED_D3.0mm_Clear
- D3: value (none) -> 5V LED; footprint (none) -> LED_THT:LED_D3.0mm_Clear
- J5: value (none) -> Power In; footprint (none) -> TerminalBlock_MetzConnect:TerminalBlock_MetzConnect_Type701_RT11L02HGLU_1x02_P6.35mm_Horizontal
- J6: value (none) -> Expansion Header; footprint (none) -> Connector_IDC:IDC-Header_2x20_P2.54mm_Vertical
- J7: value (none) -> v4 Input; footprint (none) -> 302-S241:OST_302-S241
- R1: value (none) -> 2.2K; footprint (none) -> Resistor_THT:R_Axial_DIN0207_L6.3mm_D2.5mm_P7.62mm_Horizontal
- R2: value (none) -> 220; footprint (none) -> Resistor_THT:R_Axial_DIN0207_L6.3mm_D2.5mm_P7.62mm_Horizontal
